File: hardware/volcon.sch (KiCad schematic (older format))
At the start: 21 parts, among them J1 usb-c_2.0, J2 AVR-ISP-6, J3 4-Pin, Q1 NPN, Q2 NPN, U1 ATmega32U4-AU, Y1 16MHz

Commit message: Minor adjustments, clean-up and comments.  Generated schematic pdf for repo.
Other:
- note added: "2021-02-07"
- note added: "Changes from revision 1:\n- KiCAD instead of Eagle.\n- ATmega32u4 instead of AT90usb162.\n- Removed serial connector.\n- Removed reset push-button.\n- SMD instead of through-hole components.\n- USB-C connector instead of USB-B."
- note added: "volcon"
- note removed: "2021-01-26"
- note removed: "VOLCON"
Changed lines of the file:
@@
 NoConn ~ 2700 3500
 Text Notes 7400 7500 0    79   ~ 0
-VOLCON
+volcon
 Text Notes 10600 7650 0    79   ~ 0
 2
 Text Notes 8150 7650 0    79   ~ 0
-2021-01-26
+2021-02-07
 Wire Notes Line
 	4950 4500 4950 6650
@@
 Wire Notes Line
 	9950 5650 8650 5650
+Text Notes 7000 7100 0    50   ~ 0
+Changes from revision 1:\n- KiCAD instead of Eagle.\n- ATmega32u4 instead of AT90usb162.\n- Removed serial connector.\n- Removed reset push-button.\n- SMD instead of through-hole components.\n- USB-C connector instead of USB-B.
 $EndSCHEMATC
